Commit message: Add robust autonomous pick-and-place workflow

File: src/yzbot/mybot_description/urdf/camera_gazebo.xacro (robot description, xacro)
@@ -30,5 +30,7 @@
         <gazebo reference="${prefix}_link">
             <sensor type="camera" name="camera_node">
-                <update_rate>30.0</update_rate>
+                <!-- 15 Hz is sufficient for the visual servo and avoids
+                     overloading Ogre/D3D12 under Gazebo Classic on WSL. -->
+                <update_rate>15.0</update_rate>
                 <camera name="head">
                     <horizontal_fov>1.3962634</horizontal_fov>

File: src/yzbot/mybot_description/urdf/large_base_gazebo.xacro (robot description, xacro)
@@ -16,6 +16,9 @@
         <gazebo reference="${prefix}_wheel_link">
             <material>Gazebo/Gray</material>
-            <mu1>100000.0</mu1>
-            <mu2>100000.0</mu2>
+            <!-- Keep ODE contact constraints well-conditioned. Extremely large
+                 friction values can inject explosive impulses when a wheel or
+                 caster catches an obstacle, launching the whole robot. -->
+            <mu1>2.0</mu1>
+            <mu2>2.0</mu2>
         </gazebo>
     </xacro:macro>
@@ -38,5 +41,9 @@
             <left_joint>left_wheel_joint</left_joint>
             <right_joint>right_wheel_joint</right_joint>
-            <wheel_separation>${wheel_joint_y*2}</wheel_separation>
+            <!-- Wheel joint origins are at y=+/-(base_width+wheel_length)/2,
+                 so the physical centre-to-centre track is 0.370 m.  The old
+                 wheel_joint_y*2 value was 0.760 m and made commanded turns
+                 roughly twice as aggressive as the real chassis geometry. -->
+            <wheel_separation>${base_width+wheel_length}</wheel_separation>
             <wheel_diameter>${2*wheel_radius}</wheel_diameter>
             <max_wheel_torque>10</max_wheel_torque>

File: src/yzbot/mybot_description/urdf/rgbd_gazebo.xacro (robot description, xacro)
@@ -13,6 +13,8 @@
             </visual>
             <collision>
+                <!-- Match the physical housing. The former 0.30 m-wide box
+                     could contact the floor/object while the arm was folded. -->
                 <geometry>
-                    <box size="0.07 0.3 0.09" />
+                    <box size="0.15 0.04 0.04" />
                 </geometry>
             </collision>
@@ -26,6 +28,8 @@
         <gazebo reference="${prefix}_link">
             <sensor type="depth" name="${prefix}">
-                <always_on>true</always_on>
-                <update_rate>15.0</update_rate>
+                <!-- This depth stream is not used by fixed pick/place. Keep it
+                     demand-driven and light to prevent WSL D3D12 device loss. -->
+                <always_on>false</always_on>
+                <update_rate>5.0</update_rate>
                 <pose>0 0 0 0 0 0</pose>
                 <camera name="camera">

Commit message: Snapshot the verified competition build: two 5/5 rounds at 294.8/294.9 s
Accumulated work from the 2026-10-08..13 sessions plus this session's fixes,
committed as one verified snapshot. At this revision: 188 tests pass / 3
skipped, pyflakes clean, and two full competition rounds completed 5/5 in
294.8 s and 294.9 s.

Fixes carried in this snapshot:

- Cube centre of mass. <inertial><pose> held each cube's world x,y, so the
  centre of mass sat 6.4-13 m outside a 3 cm cube and the blocks drifted and
  rotated on their own. Restored to 0 0 0. A/B with gzserver alone over 45 s:
  0.2644 m of drift and 2.914 rad of rotation before, exactly 0.0000 m and
  0.000 rad after.
- tools/show_positions.py --write-back wrote world coordinates into every
  <pose> in the model block, including the link-relative inertial pose, which
  is how the cubes were corrupted. It now shields <inertial> blocks; the
  state-block link pose, which is what Gazebo restores, is still written.
- Pickup poses. config/fixed_joint_pick_place.yaml and config/profiles/
  executor_fast.yaml still carried the moved-layout values. The launch loads
  the profile by default, so the robot drove to handoff points up to 3 m from
  the cube and the camera never saw it (vision_align 33-41 s per cube). Both
  files now match the reverted layout: vision_align 8-12 s.
- zone_slot_offsets. The +/-0.16 y slots left only 0.075 m of the 0.235 m
  acceptance half-width against a systematic 0.02-0.08 m placement error; four
  slot-3 deliveries had <=18 mm of margin and one missed the zone by 9 mm.
  Pulled in to +/-0.12: budget 0.115 m, first measured margin +0.094 m.
- Cube layout reverted to the committed original; the moved layout never
  completed a round (0/14 recorded on 2026-10-12) and is preserved as
  worlds/offic_room_moved.world.

New here: config/profiles (the fast profile the launch defaults to),
scripts/moving_obstacles.py, the mybot test suite, mybot_velocity_smoother_trace,
the navigation UDP/trace experiment launches, the world variants, tools/, and
the 启动流程.md operating guide.

File: src/yzbot/mybot_description/urdf/camera_gazebo.xacro (robot description, xacro)
@@ -1,4 +1,6 @@
 <?xml version="1.0"?>
 <robot xmlns:xacro="http://www.ros.org/wiki/xacro" name="camera">
+    <xacro:arg name="camera_update_rate" default="10.0" />
+    <xacro:property name="camera_update_rate" value="$(arg camera_update_rate)" />
     <xacro:macro name="mipi_camera" params="prefix:=camera">
         <!-- Create camera reference frame -->
@@ -34,5 +36,5 @@
                      added Ogre/D3D12 render load, and rendering is what caps
                      the whole simulation at RTF ~0.2 on this WSL host. -->
-                <update_rate>10.0</update_rate>
+                <update_rate>${camera_update_rate}</update_rate>
                 <camera name="head">
                     <horizontal_fov>1.3962634</horizontal_fov>
